File: ubs3_hub.kicad_sch (KiCad schematic)
At the start: 64 parts, among them J1 USB_C_Receptacle, J2 USB_C_Receptacle, J3 USB3_A, J4 USB3_A, J5 USB3_A, U2 CH213K, U3 CH217K, U4 CH217K, U5 CH217K, U6 CH217K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

Commit message: placement finished, power layout ok
Parts:
- removed C15, C17, C18, C19: 22u/25V, Capacitor_SMD:CP_Elec_5x5.4, symbol Device:C_Polarized_Small
- added C15, C17, C18, C36: 22u, Capacitor_SMD:C_0805_2012Metric, symbol Device:C
- added H1, H2, H3, H4: MountingHole_Pad, MountingHole:MountingHole_3.2mm_M3_Pad_Via, symbol Mechanical:MountingHole_Pad
Connections:
- net GND: now also C15.2, C17.2, C18.2, C36.2, H1.1, H2.1, H3.1, H4.1
- net VBUS_OUT1: now also C15.1
- net VBUS_OUT2: now also C17.1
- net VBUS_OUT3: now also C36.1
- net VBUS_OUT4: now also C18.1

Commit message: Layout in progress
Connections:
- net P1C_SS_RX_N: now also U1.20 (P2C_SS_RXA); no longer U1.21 (P2C_SS_RXB)
- net P1C_SS_RX_P: now also U1.21 (P2C_SS_RXB); no longer U1.20 (P2C_SS_RXA)
- net P1_SS_TXC_N: now also C3.1, U1.16 (P2_SS_TXA); no longer C4.1, U1.15 (P2_SS_TXB)
- net P1_SS_TXC_P: now also C4.1, U1.15 (P2_SS_TXB); no longer C3.1, U1.16 (P2_SS_TXA)
- net P1_SS_TX_N: now also C3.2; no longer C4.2
- net P1_SS_TX_P: now also C4.2; no longer C3.2
- net P2_SS_TXC_N: now also C9.1, U1.11 (P3_SS_TXA); no longer C10.1, U1.10 (P3_SS_TXB)
- net P2_SS_TXC_P: now also C10.1, U1.10 (P3_SS_TXB); no longer C9.1, U1.11 (P3_SS_TXA)
- net P2_SS_TX_N: now also C9.2; no longer C10.2
- net P2_SS_TX_P: now also C10.2; no longer C9.2
- net P3_SS_RX_N: now also U1.5 (P4_SS_RXA); no longer U1.4 (P4_SS_RXB)
- net P3_SS_RX_P: now also U1.4 (P4_SS_RXB); no longer U1.5 (P4_SS_RXA)
- net P3_SS_TXC_N: now also C11.1, U1.2 (P4_SS_TXA); no longer C12.1, U1.1 (P4_SS_TXB)
- net P3_SS_TXC_P: now also C12.1, U1.1 (P4_SS_TXB); no longer C11.1, U1.2 (P4_SS_TXA)
- net P3_SS_TX_N: now also C11.2; no longer C12.2
- net P3_SS_TX_P: now also C12.2; no longer C11.2
- net P4_SS_RX_N: now also U1.68 (UP_SS_RXA); no longer U1.67 (UP_SS_RXB)
- net P4_SS_RX_P: now also U1.67 (UP_SS_RXB); no longer U1.68 (UP_SS_RXA)
- net P4_SS_TXC_N: now also C13.1, U1.65 (UP_SS_TXA); no longer C14.1, U1.64 (UP_SS_TXB)
- net P4_SS_TXC_P: now also C14.1, U1.64 (UP_SS_TXB); no longer C13.1, U1.65 (UP_SS_TXA)
- net P4_SS_TX_N: now also C13.2; no longer C14.2
- net P4_SS_TX_P: now also C14.2; no longer C13.2
- net UPC_SS_TXC_N: now also C5.1, U1.51 (P1C_SS_TXA); no longer C6.1, U1.50 (P1C_SS_TXB)
- net UPC_SS_TXC_P: now also C6.1, U1.50 (P1C_SS_TXB); no longer C5.1, U1.51 (P1C_SS_TXA)
- net UPC_SS_TX_N: now also C5.2; no longer C6.2
- net UPC_SS_TX_P: now also C6.2; no longer C5.2
- net UP_SS_RX_N: now also U1.55 (P1_SS_RXA); no longer U1.56 (P1_SS_RXB)
- net UP_SS_RX_P: now also U1.56 (P1_SS_RXB); no longer U1.55 (P1_SS_RXA)
Changed lines of the file:
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@@
 	)
 	(label "P1_SS_TXC_N"
-		(at 160.02 182.88 180)
+		(at 160.02 180.34 180)
 		(effects
 			(font
@@
 	)
 	(label "P1C_SS_RX_P"
-		(at 163.83 196.85 180)
+		(at 163.83 199.39 180)
 		(effects
 			(font
@@
 	)
 	(label "P4_SS_RX_P"
-		(at 49.53 158.75 0)
+		(at 49.53 161.29 0)
 		(effects
 			(font
@@
 	)
 	(label "P4_SS_TX_P"
-		(at 24.13 153.67 0)
+		(at 24.13 156.21 0)
 		(effects
 			(font
@@
 	)
 	(label "P1C_SS_RX_N"
-		(at 163.83 199.39 180)
+		(at 163.83 196.85 180)
 		(effects
 			(font
@@
 	)
 	(label "P3_SS_RX_N"
-		(at 162.56 252.73 180)
+		(at 162.56 250.19 180)
 		(effects
 			(font
@@
 	)
 	(label "P3_SS_RX_P"
-		(at 162.56 250.19 180)
+		(at 162.56 252.73 180)
 		(effects
 			(font
@@
 	)
 	(label "P2_SS_TX_P"
-		(at 187.96 218.44 180)
+		(at 187.96 220.98 180)
 		(effects
 			(font
@@
 	)
 	(label "P3_SS_TX_P"
-		(at 187.96 245.11 180)
+		(at 187.96 247.65 180)
 		(effects
 			(font
@@
 	)
 	(label "UPC_SS_TX_N"
-		(at 189.23 153.67 180)
+		(at 189.23 151.13 180)
 		(effects
 			(font
@@
 	)
 	(label "P4_SS_TXC_N"
-		(at 63.5 156.21 180)
+		(at 63.5 153.67 180)
 		(effects
 			(font
@@
 	)
 	(label "P2_SS_TX_N"
-		(at 187.96 220.98 180)
+		(at 187.96 218.44 180)
 		(effects
 			(font
@@
 	)
 	(label "P1_SS_TX_N"
-		(at 187.96 182.88 180)
+		(at 187.96 180.34 180)
 		(effects
 			(font
@@
 	)
 	(label "UPC_SS_TXC_N"
-		(at 161.29 153.67 180)
+		(at 161.29 151.13 180)
 		(effects
 			(font
@@
 	)
 	(label "P1_SS_TX_P"
-		(at 187.96 180.34 180)
+		(at 187.96 182.88 180)
 		(effects
 			(font
@@
 	)
 	(label "P1_SS_TXC_P"
-		(at 160.02 180.34 180)
+		(at 160.02 182.88 180)
 		(effects
 			(font
@@
 	)
 	(label "P2_SS_TXC_P"
-		(at 160.02 218.44 180)
+		(at 160.02 220.98 180)
 		(effects
 			(font
@@
 	)
 	(label "P3_SS_TX_N"
-		(at 187.96 247.65 180)
+		(at 187.96 245.11 180)
 		(effects
 			(font
@@
 	)
 	(label "P3_SS_TXC_P"
-		(at 160.02 245.11 180)
+		(at 160.02 247.65 180)
 		(effects
 			(font
@@
 	)
 	(label "UPC_SS_TX_P"
-		(at 189.23 151.13 180)
+		(at 189.23 153.67 180)
 		(effects
 			(font
@@
 	)
 	(label "UP_SS_RX_P"
-		(at 163.83 144.78 180)
+		(at 163.83 147.32 180)
 		(effects
 			(font
@@
 	)
 	(label "P4_SS_TX_N"
-		(at 24.13 156.21 0)
+		(at 24.13 153.67 0)
 		(effects
 			(font
@@
 	)
 	(label "UP_SS_RX_N"
-		(at 163.83 147.32 180)
+		(at 163.83 144.78 180)
 		(effects
 			(font
@@
 	)
 	(label "UPC_SS_TXC_P"
-		(at 161.29 151.13 180)
+		(at 161.29 153.67 180)
 		(effects
 			(font
@@
 	)
 	(label "P4_SS_TXC_P"
-		(at 63.5 153.67 180)
+		(at 63.5 156.21 180)
 		(effects
 			(font
@@
 	)
 	(label "P3_SS_TXC_N"
-		(at 160.02 247.65 180)
+		(at 160.02 245.11 180)
 		(effects
 			(font
@@
 	)
 	(label "P4_SS_RX_N"
-		(at 49.53 161.29 0)
+		(at 49.53 158.75 0)
 		(effects
 			(font
@@
 	)
 	(label "P2_SS_TXC_N"
-		(at 160.02 220.98 180)
-		(effects
-			(font
+		(at 160.02 218.44 180)
+		(effects
+			(font
